File: assets/media/blog/basic.brd (EAGLE design)
At the start: 36.3 x 67 mm, 61 parts

Commit message: Updated board design
Parts:
- moved U$6 17.4 mm to (51.7, 34.4), turned to 270 degrees
- moved C1 11.2 mm to (29.1, 41.2), turned to 180 degrees
- moved R1 7.16 mm to (40.5, 45.0)
- moved CAP_SENSOR_1 7.11 mm to (41.2, 41.9)
- moved CAP_SENSOR_2 5.38 mm to (42.7, 39.0)
- moved C2 3.78 mm to (27.2, 48.5), turned to 0 degrees
- moved R15 2.53 mm to (39.9, 79.3)
- moved LED24 1.65 mm to (46.7, 88.7)
- moved U$1 1.62 mm to (25.5, 34.5), turned to 90 degrees
- moved R14 1.60 mm to (43.8, 77.0)
- moved R5 1.50 mm to (25.8, 63.3)
- moved R19 1.40 mm to (27.5, 86.1)
- moved R6 1.32 mm to (29.9, 61.2)
- moved R3 1.30 mm to (23.9, 65.9)
- moved LED19 1.20 mm to (27.8, 90.9)
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Connections:
- net N$10 renamed GND
Routing:
- net GND: track 61.6 -> 67.6 mm
- net COLLECTOR: track 144.9 -> 150.6 mm
- net POWER: track 187.5 -> 184.7 mm, vias 0 -> 2
- net N$9: track 7.77 -> 5.18 mm
- net N$39: track 4.27 -> 2.10 mm
- net N$1: track 7.11 -> 5.46 mm
- net N$36: track 2.75 -> 1.20 mm
- net N$2: track 2.95 -> 1.45 mm
- net N$7: track 2.99 -> 1.69 mm
- net N$17: track 2.50 -> 1.20 mm
- net N$5: track 2.88 -> 1.68 mm
- net N$33: track 2.40 -> 1.21 mm
- net N$63: track 2.36 -> 1.27 mm
- net N$48: track 2.43 -> 1.34 mm
- net N$24: track 2.17 -> 1.17 mm
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